File: kicad/power_supply/power.sch (KiCad schematic (older format))
At the start: 12 parts

Commit message: Updated power supply schema
Parts:
- removed D?: BRIDGE, ~, symbol BRIDGE
- added C? (x4): C, ~, symbol C
- added C? (x4): CP, symbol CP
- added D?: D_SCHOTTKY, symbol D_SCHOTTKY
- added U?: 7805, symbol 7805
- added U?: 7905, symbol 7905
Connections:
- net labels added: +5V, +9V, -5V, GND, Gnd
- wire segments 29 -> 91
Other:
- moved on the sheet: C?, D?, F?, P?, T?
