File: kicad/bench_power_supply/bias_power_supply.sch (KiCad schematic (older format))
At the start: 37 parts

Commit message: added files from mint
Parts:
- removed C?: 33n, symbol C_SMALL
- added C?: 33n, symbol C_Small
- added C?: 100n, symbol C_Small
- added C? (x2): ?, symbol CP_Small
- added D? (x3): D, symbol D
- added D?: LED_SMALL, symbol Led_Small
- added R?: 500R, symbol R_Small
- added R?: 120R, symbol R_Small
- added R?: 560R, symbol R_Small
- added U?: LM317LZ, TO-92, symbol LM317LZ
- C? (x12): symbol C_SMALL -> C_Small
- C? (x3): symbol CP_SMALL -> CP_Small
- D? (x2): symbol D_SCHOTTKY_SMALL -> D_Schottky_Small
- R? (x9): symbol R_SMALL -> R_Small
- R?: value 604R -> 500R; symbol R_SMALL -> R_Small
- R?: value 200R -> 120R; symbol R_SMALL -> R_Small
Connections:
- net labels added: +9V, -9V, PwrMonitor
- wire segments 136 -> 181
Other:
- moved on the sheet: D?, L?, T?, U?
