File: kicad/bench_power_supply/pre_regulator_smps.sch (KiCad schematic (older format))
At the start: 15 parts

Commit message: commiting before install linux mint
Parts:
- removed D?: D_SMALL, symbol D_Small
- removed IC?: LTC3864, ~, symbol LTC3864
- added C1, C2, C3, C? (x2): 100n, symbol C_Small
- added C10: 470n, symbol C_Small
- added C11, C? (x2): 1u, symbol C_Small
- added C?: 330p, symbol C_Small
- added C? (x4): 10u, symbol C_Small
- added C?: 100u, symbol CP_Small
- added C?: 47u, symbol CP_Small
- added D?: STPS15H100CB, SMD, symbol D_Schottky_Small
- added D?: D_Small, symbol D_Small
- added IC1: LTC3864, symbol LTC3864
- added L1, L2: INDUCTOR_SMALL, symbol INDUCTOR_SMALL
- added L3, L? (x2): 33uH, ---, symbol INDUCTOR_SMALL
- added Q?: SUD19P06-60, TO-252, symbol SUD19P06-60
- added Q?: 2N7002, SOT-23, symbol 2N7002
- added Q?: MMBT5401, SOT-23, symbol MMBT5401
- added R2: 0R, symbol R_Small
- added R4: R010/2W, symbol R_Small
- added R? (x4): 10R, symbol R_Small
- added R?: 1k, symbol R_Small
- added R? (x3): 324k, symbol R_Small
- added R?: 4k32, symbol R_Small
- added R?: 100k, symbol R_Small
- added SH1: SH, symbol SH
- added Z1, Z2: ZENERsmall, symbol ZENERsmall
- C1: value 3m3 -> 2m2
- C5: renamed from C2; value 3m3 -> 2m2
- R1: value 18k -> 12k
- R3: renamed from R?; value 36k -> 47k
- gave numbers to parts that had none: 1
Connections:
- net labels added: DC_OUT, EARTH, Earth, POUT, PREG_OUT, SET_100%, SW
- net labels removed: POut, VBias
- wire segments 53 -> 150
Other:
- moved on the sheet: C4, C5, C6, C7, C8, C9, D1, D2, D3, D4, JP?, R1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
